File: Sound Board/A-14732-40009.brd (EAGLE design)
At the start: 160 x 100 mm, 197 parts, among them P2 AUX IN, P3 AUX OUT, P5 VOLUME, Q1 MPS3646, U1 OKI6295, U12 27C040-150, U13 27C040-150, U14 YAMAHA 2151, U15 TIL7524, U16 74LS374, U17 74LS174, U18 16L8, U19 74LS11, U2 2064, U20 74LS139, U21 74LS14, U22 74LS74, U23 74LS74, U26 74LS04, U28 YAMAHA 3012, U29 LM324D, U3 27C040, U30 MC3340, U31 HA3116, U32 TL084D, U33 TL084D, U4 6809E, U8 74LS138, U9 74LS74, Y1 3.5749MHz, Y2 8MHz

Commit message: auto regenerated, nothing useful yet
Parts:
- added C27, C34, C35, C36, C37, C38, C39, C40, C41, C42, C43: 100pF, SparkFun-Capacitors:1206-CAP
- added P1: (no value), SparkFun-Connectors:2X10_ROUND_NOSILK
- added P4: ORKIN R/W, SparkFun-Connectors:1X04_LONGPADS
- added R12, R13, R14, R15, R16, R17, R18, R19, R20, R21, R47, R49, R50, R55, R56, R57, R58: 470, resistor:R1206
- added U10, U25, U6: 26LS32A, A-14732-40009:SO16
- added U11, U24, U7: 26LS31, A-14732-40009:SO16
- added U5: 74LS374DW, 74xx-us:SO20W
- moved C65 808.0 mm to (-40.6, 153.7)
- moved R72 791.6 mm to (-35.6, 141.0)
- moved R74 783.3 mm to (-45.7, 141.0)
- moved R73 778.1 mm to (-40.6, 141.0)
- moved C92 756.5 mm to (-15.2, 153.7)
- moved C78 756.5 mm to (-127.0, 149.9)
- moved R31 751.9 mm to (-82.5, 134.6)
- moved C90 751.4 mm to (-142.2, 149.9)
- moved C32 743.0 mm to (-25.4, 149.9)
- moved C91 728.2 mm to (-147.3, 149.9)
- moved C95 662.6 mm to (-104.1, 91.4)
- moved C87 653.3 mm to (-90.2, 91.4)
- moved C86 644.4 mm to (-76.2, 91.4)
- moved C83 642.2 mm to (-34.3, 91.4)
- moved P7 642.2 mm to (-114.3, 48.3)
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Connections:
- new net N$104: U5.5, U7.7
- new net N$105: U5.6, U7.9
- new net N$106: U5.9, U7.15
- new net N$107: U11.1, U5.12
- new net N$108: U11.7, U5.15
- new net N$109: U11.9, U5.16
- new net N$110: U11.15, U5.19
- new net N$111: U11.12, U7.12
- new net N$112: R58.1, U23.12, U5.1
- new net N$98: U5.2, U7.1
- new net VCC: U24.16, U25.16, U5.20
- net 5V: now also U10.16, U11.16, U6.16, U7.16
- net ATE1: now also U23.13, U9.10, U9.12
- net CPU0: now also U5.3, U6.3
- net CPU1: now also U5.4, U6.5
- net CPU2: now also U5.7, U6.11
- net CPU3: now also U5.8, U6.13
- net CPU4: now also U10.3, U5.13
- net CPU5: now also U10.5, U5.14
- net CPU6: now also U10.11, U5.17
- net CPU7: now also U10.13, U5.18
- net GND: now also P4.1, R58.2, U10.4, U10.8, U11.4, U11.8, U24.8, U25.8, U5.10, U6.8, U7.4, U7.8
- net IRQ: now also U23.9
- net N$30: now also P4.4
- net RD-LATCH: now also U10.12
- net WR-LATCH: now also U5.11, U9.11

Commit message: autogen updated
Parts:
- R82: value 470 -> 220
- renumbered R16 to R82, R17 to R83
Connections:
- new net FFO: U24.1, U9.9
- new net N$113: U23.11, U25.13
- new net N$114: R58.1, U23.12, U24.12, U25.12, U5.1
- new net N$115: R12.1, U6.2, U7.2
- new net N$116: R19.1, U10.6, U11.6
- new net N$117: R13.1, U6.6, U7.6
- new net N$118: R20.1, U10.10, U11.10
- new net N$119: R21.1, U10.14, U11.14
- new net N$120: R82.1, R83.2, U10.1, U10.15, U10.7, U10.9, U25.1, U25.15, U25.7, U25.9, U6.1, U6.15, U6.7, U6.9
- new net N$121: C37.1, R18.2
- new net N$122: R14.1, U6.10, U7.10
- new net N$123: R15.1, U6.14, U7.14
- new net N$124: C38.1, R19.2
- new net N$125: C39.1, R20.2
- new net N$126: C40.1, R21.2
- new net N$127: R49.1, U24.6
- new net N$128: R50.1, U24.14
- new net N$129: C41.1, P1.19, R47.2
- new net N$130: C42.1, P1.15, R49.2
- new net N$131: C43.1, R50.2
- new net N$132: P1.18, R55.1, U25.2
- new net N$133: P1.17, R56.1, U25.6
- new net N$134: P1.16, R57.1, U25.10
- new net N$135: P1.13, U25.14
- new net N$136: P1.11, U24.13
- new net SND_DAT0: C27.1, P1.3, R12.2
- new net SND_DAT1: C34.1, P1.4, R13.2
- new net SND_DAT2: C35.1, P1.5, R14.2
- new net SND_DAT3: C36.1, P1.6, R15.2
- new net VIDSNDRD: U11.12, U25.11, U7.12, U9.13
- net 5V: now also R55.2, R56.2, R57.2, R82.2, U24.16, U25.16
- net ATE1: now also U24.4, U24.9, U25.4
- net GND: now also C27.2, C34.2, C35.2, C36.2, C37.2, C38.2, C39.2, C40.2, C41.2, C42.2, C43.2, P1.1, R83.1, U6.4
- net IRQ: now also U24.15
- net N$111: now also R47.1, U24.2; no longer U11.12, U7.12
- net N$112: now also R18.1, U10.2, U11.2; no longer R58.1, U23.12, U5.1
- net RD-LATCH: now also U23.10, U24.7, U6.12
- net SOFT_RES: now also U25.3
- net VCC: no longer U24.16, U25.16
- net VIDPWRON: now also U25.5

Commit message: regenerated
Parts:
- removed C27, C34: 100pF, SparkFun-Capacitors:1206-CAP
- removed R47, R49, R50, R56, R57, R58: 470, resistor:R1206
- added C44, C45: 100pF, SparkFun-Capacitors:1206-CAP
- added R16, R17: 47, resistor:R1206
- added R84, R85, R86, R91: 4.7K, resistor:R1206
- P6, P7: value (none) -> 0.156"
- R11: value 100K -> 47
- R12, R13, R14, R15, R18, R19, R20, R21: value 470 -> 47
- R4: value 4.7K -> 100
- R55: value 470 -> 100K
- moved C43 274.9 mm to (-116.8, 151.1)
- moved C42 271.7 mm to (-111.8, 151.1)
- moved C41 268.7 mm to (-106.7, 151.1)
- moved R55 260.7 mm to (-16.5, 128.3)
- moved C40 228.4 mm to (-101.6, 151.1)
- moved C37 228.4 mm to (-86.4, 151.1)
- moved C38 225.8 mm to (-91.4, 151.1)
- moved C39 223.7 mm to (-96.5, 151.1)
- moved R20 204.5 mm to (-97.8, 134.6)
- moved R21 202.0 mm to (-102.9, 134.6)
- moved R18 201.2 mm to (-87.6, 134.6)
- moved R19 198.1 mm to (-92.7, 134.6)
- moved R83 194.4 mm to (-116.8, 141.0)
- moved R82 189.0 mm to (-111.8, 141.0)
- moved R15 188.8 mm to (-72.4, 134.6)
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Connections:
- net N$135 renamed B_VIDDAV
- removed net CPU0: U1.37, U14.10, U15.11, U17.4, U5.3, U6.3
- removed net CPU1: U1.38, U14.12, U15.10, U17.14, U5.4, U6.5
- removed net CPU2: U1.39, U14.13, U15.9, U17.6, U5.7, U6.11
- removed net CPU3: U1.40, U14.14, U15.8, U5.8, U6.13
- removed net CPU4: U1.41, U10.3, U14.15, U15.7, U5.13
- removed net CPU5: U1.42, U10.5, U14.16, U15.6, U5.14
- removed net CPU6: U1.43, U10.11, U14.17, U15.5, U5.17
- removed net CPU7: U1.44, U10.13, U14.18, U15.4, U5.18
- removed net N$121: C37.1, R18.2
- removed net N$124: C38.1, R19.2
- removed net N$125: C39.1, R20.2
- removed net N$126: C40.1, R21.2
- removed net N$129: C41.1, P1.19, R47.2
- removed net N$130: C42.1, P1.15, R49.2
- removed net N$131: C43.1, R50.2
- removed net N$132: P1.18, R55.1, U25.2
- removed net N$133: P1.17, R56.1, U25.6
- removed net N$136: P1.11, U24.13
- removed net VCC: U5.20
- new net B_SND_RD: C44.1, P1.15, R20.2
- new net B_VIDRES: P1.17, R85.1, U25.6
- new net SND_DAT4: C39.1, P1.7, R15.2
- new net SND_DAT5: C40.1, P1.8, R16.2
- new net SND_DAT6: C41.1, P1.9, R17.2
- new net SND_DAT7: C42.1, P1.10, R18.2
- new net SND_DAT8: P1.18, R84.1, U25.2
- new net SND_DAV: C45.1, P1.19, R21.2
- new net SND_RDY: C43.1, P1.11, R19.2
- net +12VDEC: now also R55.2; no longer R11.2
- net 5V: now also R84.2, R85.2, R86.2, R91.2, U5.20; no longer R4.2, R55.2, R56.2, R57.2
- net AGND: no longer C3.2, C6.2, C7.2, MTG1.P1, MTG2.P1, MTG3.P1, MTG4.P1, Q1.2, U4.39
- net D0: now also U1.37, U14.10, U15.11, U17.4, U5.3, U6.3
- net D1: now also U1.38, U14.12, U15.10, U17.14, U5.4, U6.5
- net D2: now also U1.39, U14.13, U15.9, U17.6, U5.7, U6.11
- net D3: now also U1.40, U14.14, U15.8, U5.8, U6.13
- net D4: now also U1.41, U10.3, U14.15, U15.7, U5.13
- net D5: now also U1.42, U10.5, U14.16, U15.6, U5.14
- net D6: now also U1.43, U10.11, U14.17, U15.5, U5.17
- net D7: now also U1.44, U10.13, U14.18, U15.4, U5.18
- net GND: now also C3.2, C44.2, C45.2, C6.2, C7.2, MTG1.P1, MTG2.P1, MTG3.P1, MTG4.P1, Q1.2, R4.2, U4.39; no longer C27.2, C34.2, R58.2
- net N$111: now also R21.1; no longer R47.1
- net N$112: now also R15.1; no longer R18.1
- net N$114: now also R4.1; no longer R58.1
- net N$115: now also R11.1; no longer R12.1
- net N$116: now also R16.1; no longer R19.1
- net N$118: now also R17.1; no longer R20.1
- net N$119: now also R18.1; no longer R21.1
- net N$123: now also R12.1; no longer R15.1
- net N$127: now also R20.1; no longer R49.1
- net N$128: now also R19.1; no longer R50.1
- net N$134: now also R86.1; no longer R57.1
- net N$30: now also R91.1; no longer R4.1
- net N$60: now also R55.1; no longer R11.1
- net SND_DAT0: now also C35.1, R11.2; no longer C27.1, R12.2
- net SND_DAT1: now also C37.1; no longer C34.1
- net SND_DAT2: now also C38.1; no longer C35.1
- net SND_DAT3: now also R12.2; no longer R15.2
- net YAM1-OUT: no longer R44.2
- net YAM2-OUT: now also R44.2
