File: Sound Board/eagle/A-14732-40023-REPRODUCTION.brd (EAGLE design)
At the start: 162.6 x 102.9 mm, 220 parts, among them P6 POWER, P7 SPEAKER, Q1 MPS3646, U1 OKI6295, U10 26LS32A, U11 26LS31, U12 27C040-150, U13 27C040-150, U14 YAMAHA 2151, U15 TIL7524, U16 74LS374, U17 74LS174, U18 16L8, U19 74LS11, U2 2064, U20 74LS139, U21 74LS14, U22 74LS74, U23 74LS74, U24 26LS31, U25 26LS32A, U26 74LS04, U28 YAMAHA 3012, U29 LM324D, U3 27C040, U30 MC3340, U31 MB3731, U32 TL084D, U33 TL084D, U4 6809E, U5 74LS374DW, U6 26LS32A, U7 26LS31, U8 74LS138, U9 74LS74, Y1 3.5749MHz, Y2 8MHz

Commit message: another attempt, still hopeless
Parts:
- R82, R83: device resistor:R1206 -> resistor:R0805
- moved C107 28.4 mm to (148.6, 69.8), flipped to the bottom, turned to 0 degrees
- moved C32 27.3 mm to (148.6, 21.6), turned to 0 degrees
- moved C25 27.3 mm to (129.5, 73.7)
- moved C106 24.3 mm to (148.6, 73.7), flipped to the bottom, turned to 0 degrees
- moved C67 24.3 mm to (68.6, 29.2), turned to 270 degrees
- moved U24 24.2 mm to (139.7, 85.1), flipped to the bottom, turned to 180 degrees
- moved C88 23.1 mm to (108.0, 14.0), turned to 90 degrees
- moved R91 22.5 mm to (94.0, 25.4)
- moved U30 22.2 mm to (92.7, 16.5)
- moved U25 21.8 mm to (135.9, 73.7), flipped to the bottom, turned to 0 degrees
- moved R86 21.6 mm to (144.8, 76.2), flipped to the bottom, turned to 0 degrees
- moved C89 21.6 mm to (113.0, 24.1), turned to 180 degrees
- moved C105 21.6 mm to (148.6, 76.2), flipped to the bottom, turned to 180 degrees
- moved C45 19.7 mm to (153.7, 90.2), turned to 90 degrees
- moved C65 17.6 mm to (116.8, 25.4), turned to 90 degrees
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Routing:
- net GND: track 516.2 -> 1335.7 mm
- net AGND: track 0.00 -> 275.5 mm
- net 5V: track 0.00 -> 245.0 mm, vias 0 -> 1
- net D0: track 0.00 -> 130.6 mm
- net D1: track 0.00 -> 100.0 mm
- net D2: track 0.00 -> 94.5 mm
- net D3: track 0.00 -> 93.7 mm
- net /WR: track 0.00 -> 91.8 mm
- net /RD: track 0.00 -> 90.8 mm
- net RESET: track 0.00 -> 89.0 mm
- net 12V: track 0.00 -> 86.2 mm, vias 0 -> 1
- net A12: track 0.00 -> 81.7 mm
- net D6: track 0.00 -> 75.4 mm
- net A0: track 0.00 -> 70.7 mm
- net D7: track 0.00 -> 66.8 mm
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