File: Sound Board/eagle/A-14732-40023-REPRODUCTION.sch (EAGLE design)
At the start: 220 parts, among them P6 POWER, P7 SPEAKER, Q1 MPS3646, U1 OKI6295, U10 26LS32A, U11 26LS31, U12 27C040-150, U13 27C040-150, U14 YAMAHA 2151, U15 TIL7524, U16 74LS374, U17 74LS174, U18 16L8, U19 74LS11, U2 2064, U20 74LS139, U21 74LS14, U22 74LS74, U23 74LS74, U24 26LS31, U25 26LS32A, U26 74LS04, U28 YAMAHA 3012, U29 LM324D, U3 27C040, U30 MC3340, U31 MB3731, U32 TL084D, U33 TL084D, U4 6809E, U5 74LS374DW, U6 26LS32A, U7 26LS31, U8 74LS138, U9 74LS74, Y1 3.5749MHz, Y2 8MHz

Commit message: some fixes
Parts:
- R82, R83: device resistor:R-US_R1206 -> resistor:R-US_R0805
Changed lines of the file:
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@@
 <layer number="20" name="Dimension" color="15" fill="1" visible="yes" active="no"/>
 <layer number="21" name="tPlace" color="7" fill="1" visible="yes" active="no"/>
-<layer number="22" name="bPlace" color="7" fill="1" visible="yes" active="no"/>
+<layer number="22" name="bPlace" color="14" fill="1" visible="yes" active="no"/>
 <layer number="23" name="tOrigins" color="15" fill="1" visible="yes" active="no"/>
 <layer number="24" name="bOrigins" color="15" fill="1" visible="yes" active="no"/>
@@
 <layer number="49" name="Reference" color="7" fill="1" visible="yes" active="no"/>
 <layer number="50" name="dxf" color="7" fill="1" visible="yes" active="no"/>
-<layer number="51" name="tDocu" color="7" fill="1" visible="yes" active="no"/>
+<layer number="51" name="tDocu" color="6" fill="1" visible="yes" active="no"/>
 <layer number="52" name="bDocu" color="7" fill="1" visible="yes" active="no"/>
 <layer number="53" name="tGND_GNDA" color="7" fill="9" visible="yes" active="no"/>
@@
 <part name="R14" library="SparkFun-Passives" deviceset="RESISTOR" device="0805-RES" value="47"/>
 <part name="R12" library="SparkFun-Passives" deviceset="RESISTOR" device="0805-RES" value="47"/>
-<part name="R82" library="resistor" deviceset="R-US_" device="R1206" value="220"/>
-<part name="R83" library="resistor" deviceset="R-US_" device="R1206" value="470"/>
+<part name="R82" library="resistor" deviceset="R-US_" device="R0805" value="220"/>
+<part name="R83" library="resistor" deviceset="R-US_" device="R0805" value="470"/>
 <part name="C39" library="SparkFun-Passives" deviceset="CAP" device="0805" value="100pF">
 <attribute name="VOLTAGE" value="50V"/>
